File: can.kicad_sch (KiCad schematic)
At the start: 11 parts, among them U4 SN65HVD230

Commit message: Pre-Initial review
Parts:
- JP1: footprint (none) -> Jumper:SolderJumper-2_P1.3mm_Open_RoundedPad1.0x1.5mm
- R28: value 10k -> 0
Changed lines of the file:
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@@
       (effects (font (size 1.27 1.27)) (justify left))
     )
-    (property "Value" "10k" (id 1) (at 118.11 96.52 0)
+    (property "Value" "0" (id 1) (at 118.11 96.52 0)
       (effects (font (size 1.27 1.27)) (justify left))
     )
@@
     (property "Reference" "JP1" (id 0) (at 157.48 82.55 0))
     (property "Value" "TermJP" (id 1) (at 157.48 85.09 0))
-    (property "Footprint" "" (id 2) (at 157.48 88.9 0)
+    (property "Footprint" "Jumper:SolderJumper-2_P1.3mm_Open_RoundedPad1.0x1.5mm" (id 2) (at 157.48 88.9 0)
       (effects (font (size 1.27 1.27)) hide)
     )
