File: usb-uart.kicad_sch (KiCad schematic)
At the start: 16 parts, among them J3 USB_C_Receptacle_USB2.0, U6 SC4216H, U7 LTC4411

Commit message: 2nd iteration to be reviewed
Parts:
- removed C20, C25: 10uF, Capacitor_SMD:C_0603_1608Metric, symbol Device:C_Small
- removed C23: 4.7uF, Capacitor_SMD:C_0603_1608Metric, symbol Device:C_Small
- removed R24: 56k, Resistor_SMD:R_0402_1005Metric, symbol Device:R_Small
- removed R25: 10k, Resistor_SMD:R_0402_1005Metric, symbol Device:R_Small
- removed U6: SC4216H, iclr:SOIC127P599X175-9N, symbol iclr:RT9025-25GSP
- removed U7: LTC4411, Package_TO_SOT_SMD:SOT-23-5, symbol iclr:LTC4411
- J3: footprint Connector_USB:USB_C_Receptacle_GCT_USB4085 -> iclr:USB_C_Receptacle_Palconn_UTC16-G
- renumbered D4 to D1, R15 to R12, R16 to R13, R18 to R14, TP17 to TP3, TP18 to TP4, TP19 to TP5
Connections:
- no-connect marks 5 -> 2

Commit message: 3rd iteration
Parts:
- USBLED1: footprint LED_SMD:LED_0603_1608Metric -> LED_SMD:LED_0402_1005Metric
Changed lines of the file:
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@@
       (effects (font (size 1.27 1.27)))
     )
-    (property "Footprint" "LED_SMD:LED_0603_1608Metric" (at 162.56 92.71 90)
+    (property "Footprint" "LED_SMD:LED_0402_1005Metric" (at 162.56 92.71 90)
       (effects (font (size 1.27 1.27)) hide)
     )

Commit message: rerouted spi bus and changed NAND
Parts:
- removed TP5: TestPoint, TestPoint:TestPoint_Pad_D1.0mm, symbol Connector:TestPoint
Changed lines of the file:
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@@
-    (stroke (width 0) (type default))
-  )
-  (wire (pts (xy 44.45 109.22) (xy 52.07 109.22))
     (stroke (width 0) (type default))
   )
@@
   )
   (label "Data-" (at 116.84 102.87 0) (fields_autoplaced)
-    (effects (font (size 1.27 1.27)) (justify left bottom))
-  )
-  (label "VBUS" (at 44.45 109.22 0) (fields_autoplaced)
     (effects (font (size 1.27 1.27)) (justify left bottom))
   )
@@
     (pin "1")
     (instances
-      (project "Altimeter"
+      (project "Altimeter_super_thin"
         (path "/7db990e4-92e1-4f99-b4d2-435bbec1ba83/00000000-0000-0000-0000-000061925999"
           (reference "#PWR035") (unit 1)
@@
     (pin "2")
     (instances
-      (project "Altimeter"
+      (project "Altimeter_super_thin"
         (path "/7db990e4-92e1-4f99-b4d2-435bbec1ba83/00000000-0000-0000-0000-000061925999"
           (reference "R13") (unit 1)
@@
     (pin "2")
     (instances
-      (project "Altimeter"
+      (project "Altimeter_super_thin"
         (path "/7db990e4-92e1-4f99-b4d2-435bbec1ba83/00000000-0000-0000-0000-000061925999"
           (reference "R12") (unit 1)
@@
     (pin "1")
     (instances
-      (project "Altimeter"
+      (project "Altimeter_super_thin"
         (path "/7db990e4-92e1-4f99-b4d2-435bbec1ba83/00000000-0000-0000-0000-000061925999"
           (reference "#PWR033") (unit 1)
@@
     (pin "S1")
     (instances
-      (project "Altimeter"
+      (project "Altimeter_super_thin"
         (path "/7db990e4-92e1-4f99-b4d2-435bbec1ba83/00000000-0000-0000-0000-000061925999"
           (reference "J3") (unit 1)
@@
     (pin "1")
     (instances
-      (project "Altimeter"
+      (project "Altimeter_super_thin"
         (path "/7db990e4-92e1-4f99-b4d2-435bbec1ba83/00000000-0000-0000-0000-000061925999"
           (reference "#PWR036") (unit 1)
@@
     (pin "4")
     (instances
-      (project "Altimeter"
+      (project "Altimeter_super_thin"
         (path "/7db990e4-92e1-4f99-b4d2-435bbec1ba83/00000000-0000-0000-0000-000061925999"
           (reference "D1") (unit 1)
@@
     (pin "1")
     (instances
-      (project "Altimeter"
+      (project "Altimeter_super_thin"
         (path "/7db990e4-92e1-4f99-b4d2-435bbec1ba83/00000000-0000-0000-0000-000061925999"
           (reference "#PWR034") (unit 1)
@@
     (pin "1")
     (instances
-      (project "Altimeter"
+      (project "Altimeter_super_thin"
         (path "/7db990e4-92e1-4f99-b4d2-435bbec1ba83/00000000-0000-0000-0000-000061925999"
           (reference "TP3") (unit 1)
@@
     (pin "1")
     (instances
-      (project "Altimeter"
+      (project "Altimeter_super_thin"
         (path "/7db990e4-92e1-4f99-b4d2-435bbec1ba83/00000000-0000-0000-0000-000061925999"
           (reference "TP4") (unit 1)
@@
     )
   )
-  (symbol (lib_id "Connector:TestPoint") (at 52.07 109.22 270) (unit 1)
-    (in_bom yes) (on_board yes) (dnp no)
-    (property "Reference" "TP5" (at 56.8452 108.0516 90)
-      (effects (font (size 1.27 1.27)) (justify left))
-    )
-    (property "Value" "TestPoint" (at 56.8452 110.363 90)
-      (effects (font (size 1.27 1.27)) (justify left))
-    )
-    (property "Footprint" "TestPoint:TestPoint_Pad_D1.0mm" (at 52.07 114.3 0)
-      (effects (font (size 1.27 1.27)) hide)
-    )
-    (property "Datasheet" "~" (at 52.07 114.3 0)
-      (effects (font (size 1.27 1.27)) hide)
-    )
-    (pin "1")
-    (instances
-      (project "Altimeter"
-        (path "/7db990e4-92e1-4f99-b4d2-435bbec1ba83/00000000-0000-0000-0000-000061925999"
-          (reference "TP5") (unit 1)
-        )
-      )
-    )
-  )
   (symbol (lib_id "Device:LED_Small") (at 162.56 92.71 180) (unit 1)
     (in_bom yes) (on_board yes) (dnp no)
@@
     (pin "2")
     (instances
-      (project "Altimeter"
+      (project "Altimeter_super_thin"
         (path "/7db990e4-92e1-4f99-b4d2-435bbec1ba83/00000000-0000-0000-0000-000061925999"
           (reference "USBLED1") (unit 1)
@@
     (pin "2")
     (instances
-      (project "Altimeter"
+      (project "Altimeter_super_thin"
         (path "/7db990e4-92e1-4f99-b4d2-435bbec1ba83/00000000-0000-0000-0000-000061925999"
           (reference "R14") (unit 1)
@@
     (pin "1")
     (instances
-      (project "Altimeter"
+      (project "Altimeter_super_thin"
         (path "/7db990e4-92e1-4f99-b4d2-435bbec1ba83/00000000-0000-0000-0000-000061925999"
           (reference "#PWR038") (unit 1)
@@
     (pin "1")
     (instances
-      (project "Altimeter"
+      (project "Altimeter_super_thin"
         (path "/7db990e4-92e1-4f99-b4d2-435bbec1ba83/00000000-0000-0000-0000-000061925999"
           (reference "#PWR037") (unit 1)
