File: Hardware/Altimeter_super_thin.kicad_sch (KiCad schematic)
At the start: 58 parts, among them IC2 AS5F32G04SNDA-08LIN, J1 Conn_01x04_Male, J2 Conn_01x02_Male, Q1 PMV20ENR, U1 150044M155220, U2 ESP32-S3, U4 DPS310, Y1 40MHz±10ppm

Commit message: Ordering changes
Parts:
- C13, C14: value C -> 11pF
- U4: value DPS310 -> DPS368
- Y1: value 40MHz±10ppm -> R940000171
Changed lines of the file:
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@@
 			)
 		)
-		(property "Value" "DPS310"
+		(property "Value" "DPS368"
 			(at 254 44.45 0)
 			(effects
@@
 			)
 		)
-		(property "Value" "C"
+		(property "Value" "11pF"
 			(at 165.1 144.5514 90)
 			(effects
@@
 			)
 		)
-		(property "Value" "C"
+		(property "Value" "11pF"
 			(at 163.83 124.2314 90)
 			(effects
@@
 			)
 		)
-		(property "Value" "40MHz±10ppm"
+		(property "Value" "R940000171"
 			(at 152.4 124.46 90)
 			(effects
