File: Hardware/Altimeter_super_thin.kicad_pcb (KiCad board)
At the start: 4 copper layers, 54.5 x 18 mm, 101 parts, among them IC2 AS5F32G04SNDA-08LIN, J1 Conn_01x04_Male, J2 Conn_01x02_Male, J3 USB_C_Receptacle_USB2.0, J4 Conn_01x02_Male, Q1 PMV20ENR, U1 150044M155220, U10 MAX77827AEFD+T, U11 SC4215, U2 ESP32-S3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

Commit message: Ordering changes
Parts:
- added G***: LOGO, LOGO, B.Cu at (125.5, 88.8)
- R14: value 470 -> 5.1k
- U4: value DPS310 -> DPS368
Routing:
- net /Data+: track 22.3 -> 23.6 mm
- net /Data-: track 24.3 -> 24.9 mm
- net /MISO: track 31.7 -> 31.1 mm
- net GND: track 18.6 -> 19.1 mm
Other:
- board text added: "+"
- board text added: "-"
- board text added: "BATT IN"
- board text added: "BOOT"
- board text added: "BUZZER"
- board text added: "Designed By Jack Crane Electronics Team 2024"
- board text added: "EN"
- board text removed: "Designed By Jack Crane Electronics Team 2023"

Commit message: Regenerated production files to add RAE logo
Parts:
- added G***: LOGO, iclr:rae_logo_4mm, F.Cu at (85.3, 93.9)
Other:
- board text added: "JLCJLCJLCJLC"
